File: bms_monitor.kicad_sch (KiCad schematic)
At the start: 22 parts, among them J1 Conn_01x02, J13 Conn_ARM_JTAG_SWD_10, J2 Conn_01x02, J3 Conn_01x02, J4 Conn_01x02, U1 STM32L432KBUx, U2 MCP1812AT-033-TT, U3 DSC61XX, U4 TFBS4652

Commit message: pre production
- footprints change
Parts:
- C1, C2: footprint Capacitor_SMD:C_1206_3216Metric -> Capacitor_SMD:C_1210_3225Metric

Commit message: pre production
footprint change
Parts:
- removed J13: Conn_ARM_JTAG_SWD_10, Connector_PinHeader_1.27mm:PinHeader_2x05_P1.27mm_Vertical, symbol Connector:Conn_ARM_JTAG_SWD_10
- added J14: 5V, Connector_PinHeader_2.54mm:PinHeader_1x02_P2.54mm_Vertical, symbol Connector_Generic:Conn_01x02
- added J15: Conn_ST_STDC14, lib:SAMTEC_FTSH-107-01-L-DV-K-TR, symbol Connector:Conn_ST_STDC14
Connections:
- net +3.3V: now also J15.3 (VCC)
- net +5V: now also J14.1 (Pin_1)
- net GND: now also J14.2 (Pin_2), J15.11 (GNDDetect), J15.5 (GND), J15.7 (GND)
- net SWCLK: now also J15.6 (JCLK/SWCLK)
- net SWDIO: now also J15.4 (JTMS/SWDIO)
- net SWO: now also J15.8 (JTDO/SWO)
- net TDI: now also J15.10 (JTDI/NC)
- net ~{RESET}: now also J15.12 (~{RST})
Other:
- note added: "Programming PWR"
- moved on the sheet: J1, J2, J3, J4

Commit message: Addition
-Added USART 2 to Programming connector
Connections:
- net UART2_RX: now reaches J15.13 (VCP_RX)
- net UART2_RX: now also U1.9 (PA3)
- net UART2_TX: now reaches J15.14 (VCP_TX)
- net UART2_TX: now also U1.8 (PA2)
Other:
- moved on the sheet: J15
Changed lines of the file:
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@@
     (comment 1 "Filippo Volpe")
   )
-  (junction (at 138.43 138.43) (diameter 0) (color 0 0 0 0)
+  (junction (at 140.97 128.27) (diameter 0) (color 0 0 0 0)
   )
   (junction (at 203.2 85.09) (diameter 0) (color 0 0 0 0)
@@
     (stroke (width 0) (type default) (color 0 0 0 0))
   )
-  (wire (pts (xy 151.13 106.68) (xy 163.83 106.68))
+  (wire (pts (xy 153.67 96.52) (xy 166.37 96.52))
     (stroke (width 0) (type default) (color 0 0 0 0))
   )
@@
     (stroke (width 0) (type default) (color 0 0 0 0))
   )
-  (wire (pts (xy 135.89 138.43) (xy 138.43 138.43))
+  (wire (pts (xy 138.43 128.27) (xy 140.97 128.27))
     (stroke (width 0) (type default) (color 0 0 0 0))
   )
@@
     (stroke (width 0) (type default) (color 0 0 0 0))
   )
-  (wire (pts (xy 135.89 137.16) (xy 135.89 138.43))
+  (wire (pts (xy 138.43 127) (xy 138.43 128.27))
     (stroke (width 0) (type default) (color 0 0 0 0))
   )
@@
     (stroke (width 0) (type default) (color 0 0 0 0))
   )
+  (wire (pts (xy 215.9 96.52) (xy 228.6 96.52))
+    (stroke (width 0) (type default) (color 0 0 0 0))
+  )
   (wire (pts (xy 29.21 74.93) (xy 29.21 69.85))
     (stroke (width 0) (type default) (color 0 0 0 0))
   )
-  (wire (pts (xy 151.13 111.76) (xy 163.83 111.76))
+  (wire (pts (xy 153.67 101.6) (xy 166.37 101.6))
     (stroke (width 0) (type default) (color 0 0 0 0))
   )
@@
     (stroke (width 0) (type default) (color 0 0 0 0))
   )
+  (wire (pts (xy 153.67 121.92) (xy 166.37 121.92))
+    (stroke (width 0) (type default) (color 0 0 0 0))
+  )
   (wire (pts (xy 63.5 111.76) (xy 68.58 111.76))
     (stroke (width 0) (type default) (color 0 0 0 0))
@@
     (stroke (width 0) (type default) (color 0 0 0 0))
   )
-  (wire (pts (xy 151.13 114.3) (xy 163.83 114.3))
+  (wire (pts (xy 153.67 104.14) (xy 166.37 104.14))
     (stroke (width 0) (type default) (color 0 0 0 0))
   )
@@
     (stroke (width 0) (type default) (color 0 0 0 0))
   )
+  (wire (pts (xy 215.9 99.06) (xy 228.6 99.06))
+    (stroke (width 0) (type default) (color 0 0 0 0))
+  )
   (wire (pts (xy 77.47 43.18) (xy 64.77 43.18))
     (stroke (width 0) (type default) (color 0 0 0 0))
@@
     (stroke (width 0) (type default) (color 0 0 0 0))
   )
-  (wire (pts (xy 151.13 116.84) (xy 163.83 116.84))
+  (wire (pts (xy 153.67 106.68) (xy 166.37 106.68))
     (stroke (width 0) (type default) (color 0 0 0 0))
   )
@@
     (stroke (width 0) (type default) (color 0 0 0 0))
   )
-  (wire (pts (xy 138.43 139.7) (xy 138.43 138.43))
+  (wire (pts (xy 140.97 129.54) (xy 140.97 128.27))
     (stroke (width 0) (type default) (color 0 0 0 0))
   )
@@
     (stroke (width 0) (type default) (color 0 0 0 0))
   )
-  (wire (pts (xy 138.43 137.16) (xy 138.43 138.43))
+  (wire (pts (xy 140.97 127) (xy 140.97 128.27))
     (stroke (width 0) (type default) (color 0 0 0 0))
   )
@@
     (stroke (width 0) (type default) (color 0 0 0 0))
   )
-  (wire (pts (xy 138.43 100.33) (xy 138.43 101.6))
+  (wire (pts (xy 140.97 90.17) (xy 140.97 91.44))
     (stroke (width 0) (type default) (color 0 0 0 0))
   )
@@
     (stroke (width 0) (type default) (color 0 0 0 0))
   )
-  (wire (pts (xy 151.13 119.38) (xy 163.83 119.38))
+  (wire (pts (xy 153.67 109.22) (xy 166.37 109.22))
     (stroke (width 0) (type default) (color 0 0 0 0))
   )
@@
   )
   (wire (pts (xy 24.13 101.6) (xy 34.29 101.6))
+    (stroke (width 0) (type default) (color 0 0 0 0))
+  )
+  (wire (pts (xy 153.67 119.38) (xy 166.37 119.38))
     (stroke (width 0) (type default) (color 0 0 0 0))
   )
@@
     (effects (font (size 1.27 1.27)) (justify left bottom))
   )
-  (label "SWDIO" (at 163.83 114.3 180)
+  (label "SWDIO" (at 166.37 104.14 180)
     (effects (font (size 1.27 1.27)) (justify right bottom))
   )
@@
     (effects (font (size 1.27 1.27)) (justify left bottom))
   )
+  (label "UART2_TX" (at 166.37 121.92 180)
+    (effects (font (size 1.27 1.27)) (justify right bottom))
+  )
   (label "STACK_A_IB-" (at 45.72 179.07 0)
     (effects (font (size 1.27 1.27)) (justify left bottom))
@@
     (effects (font (size 1.27 1.27)) (justify right bottom))
   )
+  (label "UART2_RX" (at 166.37 119.38 180)
+    (effects (font (size 1.27 1.27)) (justify right bottom))
+  )
   (label "STACK_B_IB+" (at 77.47 45.72 180)
     (effects (font (size 1.27 1.27)) (justify right bottom))
   )
-  (label "~{RESET}" (at 163.83 106.68 180)
+  (label "~{RESET}" (at 166.37 96.52 180)
     (effects (font (size 1.27 1.27)) (justify right bottom))
   )
@@
     (effects (font (size 1.27 1.27)) (justify left bottom))
   )
-  (label "TDI" (at 163.83 119.38 180)
+  (label "TDI" (at 166.37 109.22 180)
     (effects (font (size 1.27 1.27)) (justify right bottom))
   )
@@
     (effects (font (size 1.27 1.27)) (justify right bottom))
   )
-  (label "SWO" (at 163.83 116.84 180)
-    (effects (font (size 1.27 1.27)) (justify right bottom))
-  )
-  (label "SWCLK" (at 163.83 111.76 180)
+  (label "SWO" (at 166.37 106.68 180)
+    (effects (font (size 1.27 1.27)) (justify right bottom))
+  )
+  (label "SWCLK" (at 166.37 101.6 180)
     (effects (font (size 1.27 1.27)) (justify right bottom))
   )
@@
     (effects (font (size 1.27 1.27)) (justify right bottom))
   )
+  (label "UART2_RX" (at 228.6 99.06 180)
+    (effects (font (size 1.27 1.27)) (justify right bottom))
+  )
   (label "SCK" (at 68.58 111.76 180)
     (effects (font (size 1.27 1.27)) (justify right bottom))
@@
   (label "IA-_A" (at 26.67 109.22 0)
     (effects (font (size 1.27 1.27)) (justify left bottom))
+  )
+  (label "UART2_TX" (at 228.6 96.52 180)
+    (effects (font (size 1.27 1.27)) (justify right bottom))
   )
   (symbol (lib_id "Device:C") (at 182.88 95.25 180) (unit 1)
@@
     (pin "1")
   )
-  (symbol (lib_id "power:+3.3V") (at 138.43 100.33 0) (unit 1)
-    (in_bom yes) (on_board yes)
-    (property "Reference" "#PWR0109" (id 0) (at 138.43 104.14 0)
-      (effects (font (size 1.27 1.27)) hide)
-    )
-    (property "Value" "+3.3V" (id 1) (at 138.43 96.52 0))
-    (property "Footprint" "" (id 2) (at 138.43 100.33 0)
-      (effects (font (size 1.27 1.27)) hide)
-    )
-    (property "Datasheet" "" (id 3) (at 138.43 100.33 0)
+  (symbol (lib_id "power:+3.3V") (at 140.97 90.17 0) (unit 1)
+    (in_bom yes) (on_board yes)
+    (property "Reference" "#PWR0109" (id 0) (at 140.97 93.98 0)
+      (effects (font (size 1.27 1.27)) hide)
+    )
+    (property "Value" "+3.3V" (id 1) (at 140.97 86.36 0))
+    (property "Footprint" "" (id 2) (at 140.97 90.17 0)
+      (effects (font (size 1.27 1.27)) hide)
+    )
+    (property "Datasheet" "" (id 3) (at 140.97 90.17 0)
       (effects (font (size 1.27 1.27)) hide)
     )
@@
     (pin "2")
   )
-  (symbol (lib_id "Connector:Conn_ST_STDC14") (at 138.43 119.38 0) (unit 1)
-    (in_bom yes) (on_board yes)
-    (property "Reference" "J15" (id 0) (at 148.59 101.6 0)
+  (symbol (lib_id "Connector:Conn_ST_STDC14") (at 140.97 109.22 0) (unit 1)
+    (in_bom yes) (on_board yes)
+    (property "Reference" "J15" (id 0) (at 151.13 91.44 0)
       (effects (font (size 1.27 1.27)) (justify right))
     )
-    (property "Value" "Conn_ST_STDC14" (id 1) (at 156.21 137.16 0)
+    (property "Value" "Conn_ST_STDC14" (id 1) (at 158.75 127 0)
       (effects (font (size 1.27 1.27)) (justify right))
     )
-    (property "Footprint" "lib:SAMTEC_FTSH-107-01-L-DV-K-TR" (id 2) (at 138.43 119.38 0)
-      (effects (font (size 1.27 1.27)) hide)
-    )
-    (property "Datasheet" "https://www.st.com/content/ccc/resource/technical/document/user_manual/group1/99/49/91/b6/b2/3a/46/e5/DM00526767/files/DM00526767.pdf/jcr:content/translations/en.DM00526767.pdf" (id 3) (at 129.54 151.13 90)
+    (property "Footprint" "lib:SAMTEC_FTSH-107-01-L-DV-K-TR" (id 2) (at 140.97 109.22 0)
+      (effects (font (size 1.27 1.27)) hide)
+    )
+    (property "Datasheet" "https://www.st.com/content/ccc/resource/technical/document/user_manual/group1/99/49/91/b6/b2/3a/46/e5/DM00526767/files/DM00526767.pdf/jcr:content/translations/en.DM00526767.pdf" (id 3) (at 132.08 140.97 90)
       (effects (font (size 1.27 1.27)) hide)
     )
@@
     (pin "1")
   )
-  (symbol (lib_id "power:GND") (at 138.43 139.7 0) (unit 1)
-    (in_bom yes) (on_board yes)
-    (property "Reference" "#PWR0110" (id 0) (at 138.43 146.05 0)
-      (effects (font (size 1.27 1.27)) hide)
-    )
-    (property "Value" "GND" (id 1) (at 138.43 143.51 0))
-    (property "Footprint" "" (id 2) (at 138.43 139.7 0)
-      (effects (font (size 1.27 1.27)) hide)
-    )
-    (property "Datasheet" "" (id 3) (at 138.43 139.7 0)
-      (effects (font (size 1.27 1.27)) hide)
-    )
+  (symbol (lib_id "power:GND") (at 140.97 129.54 0) (unit 1)
+    (in_bom yes) (on_board yes)
+    (property "Reference" "#PWR0110" (id 0) (at 140.97 135.89 0)
+      (effects (font (size 1.27 1.27)) hide)
+    )
+    (property "Value" "GND" (id 1) (at 140.97 133.35 0))
+    (property "Footprint" "" (id 2) (at 140.97 129.54 0)
+      (effects (font (size 1.27 1.27)) hide)
+    )
+    (property "Datasheet" "" (id 3) (at 140.97 129.54 0)
+      (effects (font (size 1.27 1.27)) hide)
+    )

Commit message: fix
- added pmos for reverse polarity protection to prog pwr
- fixed temp connectors numbering (silkscreen)
- regenerated fabrication files
Parts:
- added Q3: PMV65XP, Package_TO_SOT_SMD:SOT-23, symbol Device:Q_PMOS_GSD
Connections:
- net +5V: now also Q3.2 (S); no longer J14.1 (Pin_1)
- net GND: now also Q3.1 (G)
- new net: J14.1 (Pin_1), Q3.3 (D)
Other:
- moved on the sheet: J14
Changed lines of the file:
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@@
+    (stroke (width 0) (type default) (color 0 0 0 0))
+  )
+  (wire (pts (xy 155.956 52.324) (xy 159.004 52.324))
     (stroke (width 0) (type default) (color 0 0 0 0))
   )
@@
     (stroke (width 0) (type default) (color 0 0 0 0))
   )
+  (wire (pts (xy 150.876 60.96) (xy 150.876 59.944))
+    (stroke (width 0) (type default) (color 0 0 0 0))
+  )
   (wire (pts (xy 200.66 135.89) (xy 200.66 137.16))
     (stroke (width 0) (type default) (color 0 0 0 0))
@@
     (stroke (width 0) (type default) (color 0 0 0 0))
   )
-  (wire (pts (xy 169.672 55.88) (xy 169.672 57.15))
+  (wire (pts (xy 141.986 54.864) (xy 141.986 60.96))
     (stroke (width 0) (type default) (color 0 0 0 0))
   )
@@
     (stroke (width 0) (type default) (color 0 0 0 0))
   )
-  (wire (pts (xy 166.116 53.34) (xy 169.672 53.34))
+  (wire (pts (xy 138.43 52.324) (xy 145.796 52.324))
     (stroke (width 0) (type default) (color 0 0 0 0))
   )
@@
     (stroke (width 0) (type default) (color 0 0 0 0))
   )
-  (wire (pts (xy 166.116 55.88) (xy 169.672 55.88))
+  (wire (pts (xy 138.43 54.864) (xy 141.986 54.864))
     (stroke (width 0) (type default) (color 0 0 0 0))
   )
@@
     (effects (font (size 1.27 1.27)) (justify left bottom))
   )
-  (text "Programming PWR" (at 159.512 50.038 0)
+  (text "Programming PWR" (at 121.666 49.276 0)
     (effects (font (size 1.27 1.27)) (justify left bottom))
   )
@@
   (label "UART2_TX" (at 228.6 96.52 180)
     (effects (font (size 1.27 1.27)) (justify right bottom))
+  )
+  (symbol (lib_id "Device:Q_PMOS_GSD") (at 150.876 54.864 90) (unit 1)
+    (in_bom yes) (on_board yes)
+    (property "Reference" "Q3" (id 0) (at 150.876 45.974 90))
+    (property "Value" "PMV65XP" (id 1) (at 150.876 48.514 90))
+    (property "Footprint" "Package_TO_SOT_SMD:SOT-23" (id 2) (at 148.336 49.784 0)
+      (effects (font (size 1.27 1.27)) hide)
+    )
+    (property "Datasheet" "" (id 3) (at 150.876 54.864 0)
+      (effects (font (size 1.27 1.27)) hide)
+    )
+    (property "Store" "https://www.mouser.it/ProductDetail/Nexperia/PMV65XP215?qs=LOCUfHb8d9vrGIOLtHQKZA%3D%3D" (id 4) (at 150.876 54.864 0)
+      (effects (font (size 1.27 1.27)) hide)
+    )
+    (property "PN" "PMV65XP,215" (id 5) (at 150.876 54.864 0)
+      (effects (font (size 1.27 1.27)) hide)
+    )
+    (pin "1")
+    (pin "2")
+    (pin "3")
   )
   (symbol (lib_id "Device:C") (at 182.88 95.25 180) (unit 1)
@@
     (pin "1")
   )
-  (symbol (lib_id "power:+5V") (at 169.672 53.34 270) (mirror x) (unit 1)
-    (in_bom yes) (on_board yes)
-    (property "Reference" "#PWR04" (id 0) (at 165.862 53.34 0)
-      (effects (font (size 1.27 1.27)) hide)
-    )
-    (property "Value" "+5V" (id 1) (at 174.752 53.34 90))
-    (property "Footprint" "" (id 2) (at 169.672 53.34 0)
-      (effects (font (size 1.27 1.27)) hide)
-    )
-    (property "Datasheet" "" (id 3) (at 169.672 53.34 0)
-      (effects (font (size 1.27 1.27)) hide)
-    )
-    (pin "1")
-  )
   (symbol (lib_id "Device:C") (at 24.13 92.71 180) (unit 1)
     (in_bom yes) (on_board yes)
@@
     (pin "1")
   )
+  (symbol (lib_id "power:GND") (at 150.876 60.96 0) (unit 1)
+    (in_bom yes) (on_board yes)
+    (property "Reference" "#PWR0106" (id 0) (at 150.876 67.31 0)
+      (effects (font (size 1.27 1.27)) hide)
+    )
+    (property "Value" "GND" (id 1) (at 150.876 64.77 0))
+    (property "Footprint" "" (id 2) (at 150.876 60.96 0)
+      (effects (font (size 1.27 1.27)) hide)
+    )
+    (property "Datasheet" "" (id 3) (at 150.876 60.96 0)
+      (effects (font (size 1.27 1.27)) hide)
+    )
+    (pin "1")
+  )
   (symbol (lib_id "power:GND") (at 219.71 83.82 0) (unit 1)
     (in_bom yes) (on_board yes)
@@
     (pin "1")
   )
-  (symbol (lib_id "Connector_Generic:Conn_01x02") (at 161.036 53.34 0) (mirror y) (unit 1)
+  (symbol (lib_id "Connector_Generic:Conn_01x02") (at 133.35 52.324 0) (mirror y) (unit 1)
     (in_bom yes) (on_board yes) (fields_autoplaced)
-    (property "Reference" "J14" (id 0) (at 158.496 53.3399 0)
-      (effects (font (size 1.27 1.27)) (justify left))
-    )
-    (property "Value" "5V" (id 1) (at 158.496 55.8799 0)
-      (effects (font (size 1.27 1.27)) (justify left))
-    )
-    (property "Footprint" "Connector_PinHeader_2.54mm:PinHeader_1x02_P2.54mm_Vertical" (id 2) (at 161.036 53.34 0)
-      (effects (font (size 1.27 1.27)) hide)
-    )
-    (property "Datasheet" "~" (id 3) (at 161.036 53.34 0)
+    (property "Reference" "J14" (id 0) (at 130.81 52.3239 0)
+      (effects (font (size 1.27 1.27)) (justify left))
+    )
+    (property "Value" "5V" (id 1) (at 130.81 54.8639 0)
+      (effects (font (size 1.27 1.27)) (justify left))
+    )
+    (property "Footprint" "Connector_PinHeader_2.54mm:PinHeader_1x02_P2.54mm_Vertical" (id 2) (at 133.35 52.324 0)
+      (effects (font (size 1.27 1.27)) hide)
+    )
+    (property "Datasheet" "~" (id 3) (at 133.35 52.324 0)
       (effects (font (size 1.27 1.27)) hide)
     )
@@
     (pin "2")
   )
-  (symbol (lib_id "power:GND") (at 169.672 57.15 0) (mirror y) (unit 1)
-    (in_bom yes) (on_board yes)
-    (property "Reference" "#PWR017" (id 0) (at 169.672 63.5 0)
-      (effects (font (size 1.27 1.27)) hide)
-    )
-    (property "Value" "GND" (id 1) (at 169.672 60.96 0))
-    (property "Footprint" "" (id 2) (at 169.672 57.15 0)
-      (effects (font (size 1.27 1.27)) hide)
-    )
-    (property "Datasheet" "" (id 3) (at 169.672 57.15 0)
+  (symbol (lib_id "power:GND") (at 141.986 60.96 0) (mirror y) (unit 1)
+    (in_bom yes) (on_board yes)
+    (property "Reference" "#PWR017" (id 0) (at 141.986 67.31 0)
+      (effects (font (size 1.27 1.27)) hide)
+    )
+    (property "Value" "GND" (id 1) (at 141.986 64.77 0))
+    (property "Footprint" "" (id 2) (at 141.986 60.96 0)
+      (effects (font (size 1.27 1.27)) hide)
+    )
+    (property "Datasheet" "" (id 3) (at 141.986 60.96 0)
       (effects (font (size 1.27 1.27)) hide)
     )
@@
     (pin "9")
   )
+  (symbol (lib_id "power:+5V") (at 159.004 52.324 270) (mirror x) (unit 1)
+    (in_bom yes) (on_board yes)
+    (property "Reference" "#PWR0105" (id 0) (at 155.194 52.324 0)
+      (effects (font (size 1.27 1.27)) hide)
+    )
+    (property "Value" "+5V" (id 1) (at 164.084 52.324 90))
+    (property "Footprint" "" (id 2) (at 159.004 52.324 0)
+      (effects (font (size 1.27 1.27)) hide)
+    )
+    (property "Datasheet" "" (id 3) (at 159.004 52.324 0)
+      (effects (font (size 1.27 1.27)) hide)
+    )
+    (pin "1")
+  )
   (symbol (lib_id "Device:C") (at 29.21 92.71 180) (unit 1)
     (in_bom yes) (on_board yes)
@@
       (reference "#PWR03") (unit 1) (value "GND") (footprint "")
     )
-    (path "/1fe265fb-1a84-4c45-92e7-50f59fee08cb"
-      (reference "#PWR04") (unit 1) (value "+5V") (footprint "")
-    )
     (path "/8633ee74-210c-4ee5-aed2-8d688468dee9"
       (reference "#PWR05") (unit 1) (value "GND") (footprint "")
@@
       (reference "#PWR0104") (unit 1) (value "+5V") (footprint "")
     )
+    (path "/b1c1e07a-51b7-48f2-9195-0393dcfa5cfc"
+      (reference "#PWR0105") (unit 1) (value "+5V") (footprint "")
+    )
+    (path "/2e4b6304-8247-4972-a806-0a0a6f2e3eb5"
+      (reference "#PWR0106") (unit 1) (value "GND") (footprint "")
+    )
     (path "/9e8e044d-840f-4911-a9ec-6064f940b10c"
       (reference "#PWR0107") (unit 1) (value "GND") (footprint "")
@@
       (reference "Q2") (unit 1) (value "NSV1C201MZ4") (footprint "Package_TO_SOT_SMD:SOT-223-3_TabPin2")
     )
+    (path "/02249555-c827-4717-b89b-3748e4f052ab"
+      (reference "Q3") (unit 1) (value "PMV65XP") (footprint "Package_TO_SOT_SMD:SOT-23")
+    )
     (path "/f6454760-ef00-4400-bda1-2718321d2678/9fbdd9db-7bbd-40b3-af15-74ac01cb2e7d"
